File: MicroSpot V2.kicad_pcb (KiCad board)
At the start: 2 copper layers, 65 x 56.2 mm, 88 parts, among them IC1 SX1255, J2 U.FL, J3 RPi, J4 WP, J5 U.FL, Q1 BSS84, U1 MCP1703Ax-330xxDB, U2 24LC256, U3 74LVC1G74DP_125, X1 TA0655A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

Commit message: Add files via upload
Parts:
- added REF**: OSHW-Logo2_7.3x6mm_SilkScreen, Symbol:OSHW-Logo2_7.3x6mm_SilkScreen, F.Cu at (160.8, 100.0)
Routing:
- net GND: track 11.8 -> 13.5 mm, vias 434 -> 435
